Commit message: The first could use but not succesful get EE pos and ori version.

File: mobile_manipulator_assets/description/urdf/ridgeback_ur5.urdf (robot description, URDF)
Before this commit: robot ridgeback, 29 links, 28 joints
Links:
- link chassis_link: geometry visual mesh filename=package://ocs2_robotic_assets/resources/mobile_manipulator/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
- link front_left_wheel_link: geometry visual mesh filename=package://ocs2_robotic_assets/resources/mobile_manipulator/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
- link front_right_wheel_link: geometry visual mesh filename=package://ocs2_robotic_assets/resources/mobile_manipulator/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
- link rear_left_wheel_link: geometry visual mesh filename=package://ocs2_robotic_assets/resources/mobile_manipulator/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
- link rear_right_wheel_link: geometry visual mesh filename=package://ocs2_robotic_assets/resources/mobile_manipulator/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
- link top_link: geometry visual mesh filename=package://ocs2_robotic_assets/resources/mobile_manipulator/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
- link ur_arm_base_link_inertia: geometry visual mesh filename=package://ocs2_robotic_assets/resources/mobile_manipulator/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
- link ur_arm_forearm_link: geometry visual mesh filename=package://ocs2_robotic_assets/resources/mobile_manipulator/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
- link ur_arm_shoulder_link: geometry visual mesh filename=package://ocs2_robotic_assets/resources/mobile_manipulator/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
- link ur_arm_upper_arm_link: geometry visual mesh filename=package://ocs2_robotic_assets/resources/mobile_manipulator/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
- link ur_arm_wrist_1_link: geometry visual mesh filename=package://ocs2_robotic_assets/resources/mobile_manipulator/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
- link ur_arm_wrist_2_link: geometry visual mesh filename=package://ocs2_robotic_assets/resources/mobile_manipulator/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
- link ur_arm_wrist_3_link: geometry visual mesh filename=package://ocs2_robotic_assets/resources/mobile_manipulator/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
