Commit message: Change file dim.

File: mobile_manipulator_assets/description/OCS2_mobile_manipulator/urdf/ridgeback_ur5.urdf (robot description, URDF)
Before this commit: robot ridgeback, 29 links, 28 joints
Links:
- link axle_link: geometry visual mesh filename=package://mobile_manipulator_assets/description/OCS2_mobile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
- link chassis_link: geometry visual mesh filename=package://mobile_manipulator_assets/description/OCS2_mobile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
- link front_cover_link: geometry visual mesh filename=package://mobile_manipulator_assets/description/OCS2_mobile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
- link front_left_wheel_link: geometry visual mesh filename=package://mobile_manipulator_assets/description/OCS2_mobile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
- link front_lights_link: geometry visual mesh filename=package://mobile_manipulator_assets/description/OCS2_mobile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
- link front_right_wheel_link: geometry visual mesh filename=package://mobile_manipulator_assets/description/OCS2_mobile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
- link front_rocker_link: geometry visual mesh filename=package://mobile_manipulator_assets/description/OCS2_mobile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
- link left_side_cover_link: geometry visual mesh filename=package://mobile_manipulator_assets/description/OCS2_mobile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
- link rear_cover_link: geometry visual mesh filename=package://mobile_manipulator_assets/description/OCS2_mobile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
- link rear_left_wheel_link: geometry visual mesh filename=package://mobile_manipulator_assets/description/OCS2_mobile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
- link rear_lights_link: geometry visual mesh filename=package://mobile_manipulator_assets/description/OCS2_mobile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
- link rear_right_wheel_link: geometry visual mesh filename=package://mobile_manipulator_assets/description/OCS2_mobile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
- link rear_rocker_link: geometry visual mesh filename=package://mobile_manipulator_assets/description/OCS2_mobile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
- link right_side_cover_link: geometry visual mesh filename=package://mobile_manipulator_assets/description/OCS2_mobile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
- link top_link: geometry visual mesh filename=package://mobile_manipulator_assets/description/OCS2_mobile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
- link ur_arm_base_link_inertia: geometry visual mesh filename=package://mobile_manipulator_assets/description/OCS2_mobile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
- link ur_arm_forearm_link: geometry visual mesh filename=package://mobile_manipulator_assets/description/OCS2_mobile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
- link ur_arm_shoulder_link: geometry visual mesh filename=package://mobile_manipulator_assets/description/OCS2_mobile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
- link ur_arm_upper_arm_link: geometry visual mesh filename=package://mobile_manipulator_assets/description/OCS2_mobile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
- link ur_arm_wrist_1_link: geometry visual mesh filename=package://mobile_manipulator_assets/description/OCS2_mobile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
- link ur_arm_wrist_2_link: geometry visual mesh filename=package://mobile_manipulator_assets/description/OCS2_mobile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
- link ur_arm_wrist_3_link: geometry visual mesh filename=package://mobile_manipulator_assets/description/OCS2_mobile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

Commit message: Fix urdf's <link> and then success use urdf2webots creat proto.

File: mobile_manipulator_assets/description/OCS2_mobile_manipulator/urdf/ridgeback_ur5.urdf (robot description, URDF)
Before this commit: robot ridgeback, 29 links, 28 joints
Links:
- removed link imu_link
- removed link mid_mount
- removed link ur_arm_base_link_inertia
- link axle_link: mass None -> 0.1
- link front_cover_link: mass None -> 0.1
- link front_lights_link: mass None -> 0.1
- link left_side_cover_link: mass None -> 0.1
- link rear_cover_link: mass None -> 0.1
- link rear_lights_link: mass None -> 0.1
- link right_side_cover_link: mass None -> 0.1
- link top_link: mass None -> 0.1
- link ur_arm_base_link: mass None -> 4.0; geometry visual mesh filename=package://mobile_manipulator_assets/description/OCS2_mobile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
Joints:
- removed joint imu_joint
- removed joint mid_mount_joint
- removed joint ur_arm_base_link-base_link_inertia
- joint arm_mount_joint: origin xyz=0 0 0 rpy=0 0 0 -> xyz=0 0 0.28 rpy=0 0 0; parent mid_mount -> base_link
- joint ur_arm_shoulder_pan_joint: parent ur_arm_base_link_inertia -> ur_arm_base_link

Commit message: Fix urdf's wheel type to continues.

File: mobile_manipulator_assets/description/OCS2_mobile_manipulator/urdf/ridgeback_ur5.urdf (robot description, URDF)
Before this commit: robot ridgeback, 26 links, 25 joints
Joints:
- joint front_left_wheel: axis (none) -> 0 1 0; type fixed -> continuous
- joint front_right_wheel: axis (none) -> 0 1 0; type fixed -> continuous
- joint rear_left_wheel: axis (none) -> 0 1 0; type fixed -> continuous
- joint rear_right_wheel: axis (none) -> 0 1 0; type fixed -> continuous

Commit message: The urdf wheel should be fixed except creat proto.

File: mobile_manipulator_assets/description/OCS2_mobile_manipulator/urdf/ridgeback_ur5.urdf (robot description, URDF)
Before this commit: robot ridgeback, 26 links, 25 joints
Joints:
- joint front_left_wheel: axis 0 1 0 -> (none); type continuous -> fixed
- joint front_right_wheel: axis 0 1 0 -> (none); type continuous -> fixed
- joint rear_left_wheel: axis 0 1 0 -> (none); type continuous -> fixed
- joint rear_right_wheel: axis 0 1 0 -> (none); type continuous -> fixed

Commit message: Change ur_arm_wrist_2_joint to webots.

File: mobile_manipulator_assets/description/OCS2_mobile_manipulator/urdf/ridgeback_ur5.urdf (robot description, URDF)
Before this commit: robot ridgeback, 26 links, 25 joints
Joints:
- joint ur_arm_wrist_2_joint: origin xyz=0 -0.09465 -1.941303950897609e-11 rpy=1.570796327 0 0 -> xyz=0 -0.09465 -1.941303950897609e-11 rpy=1.570796327 -1.570796327 0
