Commit message: change mobile_manipulator_assets to mm_assets.

File: mm_assets/description/OCS2_mobile_manipulator/urdf/ridgeback_ur5.urdf (robot description, URDF)
Before this commit: robot ridgeback, 26 links, 25 joints
Links:
- link axle_link: geometry visual mesh filename=package://mm_assets/description/OCS2_mobile_manipulator/mes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
- link chassis_link: geometry visual mesh filename=package://mm_assets/description/OCS2_mobile_manipulator/mes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
- link front_cover_link: geometry visual mesh filename=package://mm_assets/description/OCS2_mobile_manipulator/mes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
- link front_left_wheel_link: geometry visual mesh filename=package://mm_assets/description/OCS2_mobile_manipulator/mes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
- link front_lights_link: geometry visual mesh filename=package://mm_assets/description/OCS2_mobile_manipulator/mes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
- link front_right_wheel_link: geometry visual mesh filename=package://mm_assets/description/OCS2_mobile_manipulator/mes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
- link front_rocker_link: geometry visual mesh filename=package://mm_assets/description/OCS2_mobile_manipulator/mes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
- link left_side_cover_link: geometry visual mesh filename=package://mm_assets/description/OCS2_mobile_manipulator/mes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
- link rear_cover_link: geometry visual mesh filename=package://mm_assets/description/OCS2_mobile_manipulator/mes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
- link rear_left_wheel_link: geometry visual mesh filename=package://mm_assets/description/OCS2_mobile_manipulator/mes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
- link rear_lights_link: geometry visual mesh filename=package://mm_assets/description/OCS2_mobile_manipulator/mes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
- link rear_right_wheel_link: geometry visual mesh filename=package://mm_assets/description/OCS2_mobile_manipulator/mes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
- link rear_rocker_link: geometry visual mesh filename=package://mm_assets/description/OCS2_mobile_manipulator/mes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
- link right_side_cover_link: geometry visual mesh filename=package://mm_assets/description/OCS2_mobile_manipulator/mes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
- link top_link: geometry visual mesh filename=package://mm_assets/description/OCS2_mobile_manipulator/mes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
- link ur_arm_base_link: geometry visual mesh filename=package://mm_assets/description/OCS2_mobile_manipulator/mes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
- link ur_arm_forearm_link: geometry visual mesh filename=package://mm_assets/description/OCS2_mobile_manipulator/mes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
- link ur_arm_shoulder_link: geometry visual mesh filename=package://mm_assets/description/OCS2_mobile_manipulator/mes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
- link ur_arm_upper_arm_link: geometry visual mesh filename=package://mm_assets/description/OCS2_mobile_manipulator/mes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
- link ur_arm_wrist_1_link: geometry visual mesh filename=package://mm_assets/description/OCS2_mobile_manipulator/mes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
- link ur_arm_wrist_2_link: geometry visual mesh filename=package://mm_assets/description/OCS2_mobile_manipulator/mes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
- link ur_arm_wrist_3_link: geometry visual mesh filename=package://mm_assets/description/OCS2_mobile_manipulator/mes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

File: mm_assets/description/OCS2_mobile_manipulator/urdf/ridgeback_ur5_for_webots.urdf (robot description, URDF)
Before this commit: robot ridgeback, 26 links, 25 joints
Links:
- link axle_link: geometry visual mesh filename=package://mm_assets/description/OCS2_mobile_manipulator/mes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
- link chassis_link: geometry visual mesh filename=package://mm_assets/description/OCS2_mobile_manipulator/mes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
- link front_cover_link: geometry visual mesh filename=package://mm_assets/description/OCS2_mobile_manipulator/mes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
- link front_left_wheel_link: geometry visual mesh filename=package://mm_assets/description/OCS2_mobile_manipulator/mes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
- link front_lights_link: geometry visual mesh filename=package://mm_assets/description/OCS2_mobile_manipulator/mes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
- link front_right_wheel_link: geometry visual mesh filename=package://mm_assets/description/OCS2_mobile_manipulator/mes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
- link front_rocker_link: geometry visual mesh filename=package://mm_assets/description/OCS2_mobile_manipulator/mes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
- link left_side_cover_link: geometry visual mesh filename=package://mm_assets/description/OCS2_mobile_manipulator/mes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
- link rear_cover_link: geometry visual mesh filename=package://mm_assets/description/OCS2_mobile_manipulator/mes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
- link rear_left_wheel_link: geometry visual mesh filename=package://mm_assets/description/OCS2_mobile_manipulator/mes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
- link rear_lights_link: geometry visual mesh filename=package://mm_assets/description/OCS2_mobile_manipulator/mes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
- link rear_right_wheel_link: geometry visual mesh filename=package://mm_assets/description/OCS2_mobile_manipulator/mes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
- link rear_rocker_link: geometry visual mesh filename=package://mm_assets/description/OCS2_mobile_manipulator/mes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
- link right_side_cover_link: geometry visual mesh filename=package://mm_assets/description/OCS2_mobile_manipulator/mes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
- link top_link: geometry visual mesh filename=package://mm_assets/description/OCS2_mobile_manipulator/mes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
- link ur_arm_base_link: geometry visual mesh filename=package://mm_assets/description/OCS2_mobile_manipulator/mes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
- link ur_arm_forearm_link: geometry visual mesh filename=package://mm_assets/description/OCS2_mobile_manipulator/mes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
- link ur_arm_shoulder_link: geometry visual mesh filename=package://mm_assets/description/OCS2_mobile_manipulator/mes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
- link ur_arm_upper_arm_link: geometry visual mesh filename=package://mm_assets/description/OCS2_mobile_manipulator/mes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
- link ur_arm_wrist_1_link: geometry visual mesh filename=package://mm_assets/description/OCS2_mobile_manipulator/mes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
- link ur_arm_wrist_2_link: geometry visual mesh filename=package://mm_assets/description/OCS2_mobile_manipulator/mes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
- link ur_arm_wrist_3_link: geometry visual mesh filename=package://mm_assets/description/OCS2_mobile_manipulator/mes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

File: mm_assets/description/OCS2_mobile_manipulator/urdf/ridgeback_ur5_gazebo.urdf (robot description, URDF)
Before this commit: robot ridgeback, 26 links, 25 joints
Links:
- link axle_link: geometry collision mesh filename=package://mm_assets/description/OCS2_mobile_manipulator/mes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; visual mesh filename=package://mm_assets/description/OCS2_mobile_manipulator/mes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
- link chassis_link: geometry collision mesh filename=package://mm_assets/description/OCS2_mobile_manipulator/mes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; visual mesh filename=package://mm_assets/description/OCS2_mobile_manipulator/mes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
- link front_cover_link: geometry collision mesh filename=package://mm_assets/description/OCS2_mobile_manipulator/mes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; visual mesh filename=package://mm_assets/description/OCS2_mobile_manipulator/mes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
- link front_left_wheel_link: geometry collision mesh filename=package://mm_assets/description/OCS2_mobile_manipulator/mes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; visual mesh filename=package://mm_assets/description/OCS2_mobile_manipulator/mes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
- link front_lights_link: geometry collision mesh filename=package://mm_assets/description/OCS2_mobile_manipulator/mes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; visual mesh filename=package://mm_assets/description/OCS2_mobile_manipulator/mes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
- link front_right_wheel_link: geometry collision mesh filename=package://mm_assets/description/OCS2_mobile_manipulator/mes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; visual mesh filename=package://mm_assets/description/OCS2_mobile_manipulator/mes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
- link front_rocker_link: geometry collision mesh filename=package://mm_assets/description/OCS2_mobile_manipulator/mes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; visual mesh filename=package://mm_assets/description/OCS2_mobile_manipulator/mes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
- link left_side_cover_link: geometry collision mesh filename=package://mm_assets/description/OCS2_mobile_manipulator/mes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; visual mesh filename=package://mm_assets/description/OCS2_mobile_manipulator/mes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
- link rear_cover_link: geometry collision mesh filename=package://mm_assets/description/OCS2_mobile_manipulator/mes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; visual mesh filename=package://mm_assets/description/OCS2_mobile_manipulator/mes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
- link rear_left_wheel_link: geometry collision mesh filename=package://mm_assets/description/OCS2_mobile_manipulator/mes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; visual mesh filename=package://mm_assets/description/OCS2_mobile_manipulator/mes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
- link rear_lights_link: geometry collision mesh filename=package://mm_assets/description/OCS2_mobile_manipulator/mes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; visual mesh filename=package://mm_assets/description/OCS2_mobile_manipulator/mes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
- link rear_right_wheel_link: geometry collision mesh filename=package://mm_assets/description/OCS2_mobile_manipulator/mes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; visual mesh filename=package://mm_assets/description/OCS2_mobile_manipulator/mes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
- link rear_rocker_link: geometry collision mesh filename=package://mm_assets/description/OCS2_mobile_manipulator/mes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; visual mesh filename=package://mm_assets/description/OCS2_mobile_manipulator/mes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
- link right_side_cover_link: geometry collision mesh filename=package://mm_assets/description/OCS2_mobile_manipulator/mes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; visual mesh filename=package://mm_assets/description/OCS2_mobile_manipulator/mes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
- link top_link: geometry collision mesh filename=package://mm_assets/description/OCS2_mobile_manipulator/mes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; visual mesh filename=package://mm_assets/description/OCS2_mobile_manipulator/mes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
- link ur_arm_base_link: geometry collision mesh filename=package://mm_assets/description/OCS2_mobile_manipulator/mes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; visual mesh filename=package://mm_assets/description/OCS2_mobile_manipulator/mes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
- link ur_arm_forearm_link: geometry collision mesh filename=package://mm_assets/description/OCS2_mobile_manipulator/mes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; visual mesh filename=package://mm_assets/description/OCS2_mobile_manipulator/mes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
- link ur_arm_shoulder_link: geometry collision mesh filename=package://mm_assets/description/OCS2_mobile_manipulator/mes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; visual mesh filename=package://mm_assets/description/OCS2_mobile_manipulator/mes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
- link ur_arm_upper_arm_link: geometry collision mesh filename=package://mm_assets/description/OCS2_mobile_manipulator/mes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; visual mesh filename=package://mm_assets/description/OCS2_mobile_manipulator/mes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
- link ur_arm_wrist_1_link: geometry collision mesh filename=package://mm_assets/description/OCS2_mobile_manipulator/mes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; visual mesh filename=package://mm_assets/description/OCS2_mobile_manipulator/mes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
- link ur_arm_wrist_2_link: geometry collision mesh filename=package://mm_assets/description/OCS2_mobile_manipulator/mes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; visual mesh filename=package://mm_assets/description/OCS2_mobile_manipulator/mes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
- link ur_arm_wrist_3_link: geometry collision mesh filename=package://mm_assets/description/OCS2_mobile_manipulator/mes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; visual mesh filename=package://mm_assets/description/OCS2_mobile_manipulator/mes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
