Commit message: change OCS2_mobile_manipulator to ocs2_mm.

File: mm_assets/description/ocs2_mm/urdf/ridgeback_ur5.urdf (robot description, URDF)
Before this commit: robot ridgeback, 26 links, 25 joints
Links:
- link axle_link: geometry visual mesh filename=package://mm_assets/description/ocs2_mm/meshes/base/axle.stl
- link chassis_link: geometry visual mesh filename=package://mm_assets/description/ocs2_mm/meshes/base/body.stl
- link front_cover_link: geometry visual mesh filename=package://mm_assets/description/ocs2_mm/meshes/base/end-cov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
- link front_left_wheel_link: geometry visual mesh filename=package://mm_assets/description/ocs2_mm/meshes/base/wheel.s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
- link front_lights_link: geometry visual mesh filename=package://mm_assets/description/ocs2_mm/meshes/base/lights.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
- link front_right_wheel_link: geometry visual mesh filename=package://mm_assets/description/ocs2_mm/meshes/base/wheel.s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
- link front_rocker_link: geometry visual mesh filename=package://mm_assets/description/ocs2_mm/meshes/base/rocker.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
- link left_side_cover_link: geometry visual mesh filename=package://mm_assets/description/ocs2_mm/meshes/base/side-co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
- link rear_cover_link: geometry visual mesh filename=package://mm_assets/description/ocs2_mm/meshes/base/end-cov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
- link rear_left_wheel_link: geometry visual mesh filename=package://mm_assets/description/ocs2_mm/meshes/base/wheel.s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
- link rear_lights_link: geometry visual mesh filename=package://mm_assets/description/ocs2_mm/meshes/base/lights.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
- link rear_right_wheel_link: geometry visual mesh filename=package://mm_assets/description/ocs2_mm/meshes/base/wheel.s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
- link rear_rocker_link: geometry visual mesh filename=package://mm_assets/description/ocs2_mm/meshes/base/rocker.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
- link right_side_cover_link: geometry visual mesh filename=package://mm_assets/description/ocs2_mm/meshes/base/side-co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
- link top_link: geometry visual mesh filename=package://mm_assets/description/ocs2_mm/meshes/base/top.stl
- link ur_arm_base_link: geometry visual mesh filename=package://mm_assets/description/ocs2_mm/meshes/ur5/visual/b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
- link ur_arm_forearm_link: geometry visual mesh filename=package://mm_assets/description/ocs2_mm/meshes/ur5/visual/f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
- link ur_arm_shoulder_link: geometry visual mesh filename=package://mm_assets/description/ocs2_mm/meshes/ur5/visual/s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
- link ur_arm_upper_arm_link: geometry visual mesh filename=package://mm_assets/description/ocs2_mm/meshes/ur5/visual/u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
- link ur_arm_wrist_1_link: geometry visual mesh filename=package://mm_assets/description/ocs2_mm/meshes/ur5/visual/w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
- link ur_arm_wrist_2_link: geometry visual mesh filename=package://mm_assets/description/ocs2_mm/meshes/ur5/visual/w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
- link ur_arm_wrist_3_link: geometry visual mesh filename=package://mm_assets/description/ocs2_mm/meshes/ur5/visual/w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
Joints:
- joint front_left_wheel: axis 0 1 0 -> (none); type continuous -> fixed
- joint front_right_wheel: axis 0 1 0 -> (none); type continuous -> fixed
- joint rear_left_wheel: axis 0 1 0 -> (none); type continuous -> fixed
- joint rear_right_wheel: axis 0 1 0 -> (none); type continuous -> fixed
- joint ur_arm_wrist_2_joint: origin xyz=0 -0.09465 -1.941303950897609e-11 rpy=1.570796327 0 0 -> xyz=0 -0.09465 -1.941303950897609e-11 rpy=1.570796327 -1.570796327 0

File: mm_assets/description/ocs2_mm/urdf/ridgeback_ur5_for_webots.urdf (robot description, URDF)
Before this commit: robot ridgeback, 26 links, 25 joints
Links:
- link axle_link: geometry visual mesh filename=package://mm_assets/description/ocs2_mm/meshes/base/axle.stl
- link chassis_link: geometry visual mesh filename=package://mm_assets/description/ocs2_mm/meshes/base/body.stl
- link front_cover_link: geometry visual mesh filename=package://mm_assets/description/ocs2_mm/meshes/base/end-cov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
- link front_left_wheel_link: geometry visual mesh filename=package://mm_assets/description/ocs2_mm/meshes/base/wheel.s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
- link front_lights_link: geometry visual mesh filename=package://mm_assets/description/ocs2_mm/meshes/base/lights.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
- link front_right_wheel_link: geometry visual mesh filename=package://mm_assets/description/ocs2_mm/meshes/base/wheel.s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
- link front_rocker_link: geometry visual mesh filename=package://mm_assets/description/ocs2_mm/meshes/base/rocker.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
- link left_side_cover_link: geometry visual mesh filename=package://mm_assets/description/ocs2_mm/meshes/base/side-co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
- link rear_cover_link: geometry visual mesh filename=package://mm_assets/description/ocs2_mm/meshes/base/end-cov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
- link rear_left_wheel_link: geometry visual mesh filename=package://mm_assets/description/ocs2_mm/meshes/base/wheel.s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
- link rear_lights_link: geometry visual mesh filename=package://mm_assets/description/ocs2_mm/meshes/base/lights.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
- link rear_right_wheel_link: geometry visual mesh filename=package://mm_assets/description/ocs2_mm/meshes/base/wheel.s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
- link rear_rocker_link: geometry visual mesh filename=package://mm_assets/description/ocs2_mm/meshes/base/rocker.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
- link right_side_cover_link: geometry visual mesh filename=package://mm_assets/description/ocs2_mm/meshes/base/side-co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
- link top_link: geometry visual mesh filename=package://mm_assets/description/ocs2_mm/meshes/base/top.stl
- link ur_arm_base_link: geometry visual mesh filename=package://mm_assets/description/ocs2_mm/meshes/ur5/visual/b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
- link ur_arm_forearm_link: geometry visual mesh filename=package://mm_assets/description/ocs2_mm/meshes/ur5/visual/f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
- link ur_arm_shoulder_link: geometry visual mesh filename=package://mm_assets/description/ocs2_mm/meshes/ur5/visual/s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
- link ur_arm_upper_arm_link: geometry visual mesh filename=package://mm_assets/description/ocs2_mm/meshes/ur5/visual/u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
- link ur_arm_wrist_1_link: geometry visual mesh filename=package://mm_assets/description/ocs2_mm/meshes/ur5/visual/w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
- link ur_arm_wrist_2_link: geometry visual mesh filename=package://mm_assets/description/ocs2_mm/meshes/ur5/visual/w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
- link ur_arm_wrist_3_link: geometry visual mesh filename=package://mm_assets/description/ocs2_mm/meshes/ur5/visual/w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
Joints:
- joint front_left_wheel: axis (none) -> 0 1 0; type fixed -> continuous
- joint front_right_wheel: axis (none) -> 0 1 0; type fixed -> continuous
- joint rear_left_wheel: axis (none) -> 0 1 0; type fixed -> continuous
- joint rear_right_wheel: axis (none) -> 0 1 0; type fixed -> continuous
- joint ur_arm_wrist_2_joint: origin xyz=0 -0.09465 -1.941303950897609e-11 rpy=1.570796327 -1.570796327 0 -> xyz=0 -0.09465 -1.941303950897609e-11 rpy=1.570796327 0 0

File: mm_assets/description/ocs2_mm/urdf/ridgeback_ur5_gazebo.urdf (robot description, URDF)
Before this commit: robot ridgeback, 26 links, 25 joints
Links:
- link axle_link: geometry collision mesh filename=package://mm_assets/description/ocs2_mm/meshes/base/axle.stl; visual mesh filename=package://mm_assets/description/ocs2_mm/meshes/base/axle.stl
- link chassis_link: geometry collision mesh filename=package://mm_assets/description/ocs2_mm/meshes/base/body.stl; visual mesh filename=package://mm_assets/description/ocs2_mm/meshes/base/body.stl
- link front_cover_link: geometry collision mesh filename=package://mm_assets/description/ocs2_mm/meshes/base/end-cov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; visual mesh filename=package://mm_assets/description/ocs2_mm/meshes/base/end-cov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
- link front_left_wheel_link: geometry collision mesh filename=package://mm_assets/description/ocs2_mm/meshes/base/wheel.s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; visual mesh filename=package://mm_assets/description/ocs2_mm/meshes/base/wheel.s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
- link front_lights_link: geometry collision mesh filename=package://mm_assets/description/ocs2_mm/meshes/base/lights.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; visual mesh filename=package://mm_assets/description/ocs2_mm/meshes/base/lights.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
- link front_right_wheel_link: geometry collision mesh filename=package://mm_assets/description/ocs2_mm/meshes/base/wheel.s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; visual mesh filename=package://mm_assets/description/ocs2_mm/meshes/base/wheel.s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
- link front_rocker_link: geometry collision mesh filename=package://mm_assets/description/ocs2_mm/meshes/base/rocker.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; visual mesh filename=package://mm_assets/description/ocs2_mm/meshes/base/rocker.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
- link left_side_cover_link: geometry collision mesh filename=package://mm_assets/description/ocs2_mm/meshes/base/side-co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; visual mesh filename=package://mm_assets/description/ocs2_mm/meshes/base/side-co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
- link rear_cover_link: geometry collision mesh filename=package://mm_assets/description/ocs2_mm/meshes/base/end-cov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; visual mesh filename=package://mm_assets/description/ocs2_mm/meshes/base/end-cov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
- link rear_left_wheel_link: geometry collision mesh filename=package://mm_assets/description/ocs2_mm/meshes/base/wheel.s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; visual mesh filename=package://mm_assets/description/ocs2_mm/meshes/base/wheel.s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
- link rear_lights_link: geometry collision mesh filename=package://mm_assets/description/ocs2_mm/meshes/base/lights.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; visual mesh filename=package://mm_assets/description/ocs2_mm/meshes/base/lights.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
- link rear_right_wheel_link: geometry collision mesh filename=package://mm_assets/description/ocs2_mm/meshes/base/wheel.s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; visual mesh filename=package://mm_assets/description/ocs2_mm/meshes/base/wheel.s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
- link rear_rocker_link: geometry collision mesh filename=package://mm_assets/description/ocs2_mm/meshes/base/rocker.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; visual mesh filename=package://mm_assets/description/ocs2_mm/meshes/base/rocker.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
- link right_side_cover_link: geometry collision mesh filename=package://mm_assets/description/ocs2_mm/meshes/base/side-co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; visual mesh filename=package://mm_assets/description/ocs2_mm/meshes/base/side-co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
- link top_link: geometry collision mesh filename=package://mm_assets/description/ocs2_mm/meshes/base/top.stl; visual mesh filename=package://mm_assets/description/ocs2_mm/meshes/base/top.stl
- link ur_arm_base_link: geometry collision mesh filename=package://mm_assets/description/ocs2_mm/meshes/ur5/collisio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; visual mesh filename=package://mm_assets/description/ocs2_mm/meshes/ur5/visual/b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
- link ur_arm_forearm_link: geometry collision mesh filename=package://mm_assets/description/ocs2_mm/meshes/ur5/collisio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; visual mesh filename=package://mm_assets/description/ocs2_mm/meshes/ur5/visual/f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
- link ur_arm_shoulder_link: geometry collision mesh filename=package://mm_assets/description/ocs2_mm/meshes/ur5/collisio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; visual mesh filename=package://mm_assets/description/ocs2_mm/meshes/ur5/visual/s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
- link ur_arm_upper_arm_link: geometry collision mesh filename=package://mm_assets/description/ocs2_mm/meshes/ur5/collisio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; visual mesh filename=package://mm_assets/description/ocs2_mm/meshes/ur5/visual/u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
- link ur_arm_wrist_1_link: geometry collision mesh filename=package://mm_assets/description/ocs2_mm/meshes/ur5/collisio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; visual mesh filename=package://mm_assets/description/ocs2_mm/meshes/ur5/visual/w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
- link ur_arm_wrist_2_link: geometry collision mesh filename=package://mm_assets/description/ocs2_mm/meshes/ur5/collisio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; visual mesh filename=package://mm_assets/description/ocs2_mm/meshes/ur5/visual/w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
- link ur_arm_wrist_3_link: geometry collision mesh filename=package://mm_assets/description/ocs2_mm/meshes/ur5/collisio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; visual mesh filename=package://mm_assets/description/ocs2_mm/meshes/ur5/visual/w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
