Commit message: Add qz_hw.

File: mm_assets/description/ddt_mm/urdf/diablo_manipulator/robot_pinocchio.urdf (robot description, URDF)
Before this commit: robot qm, 18 links, 17 joints
Links:
- added link Ee_tray, mass 0.174621; collision mesh filename=package://mm_assets/description/ddt_mm/meshes/manipulator/l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; visual mesh filename=package://mm_assets/description/ddt_mm/meshes/manipulator/l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
Joints:
- added joint fix_Ee: type fixed, parent link6, child Ee_tray, origin xyz=0 0 0 rpy=0 0 0
