Commit message: Fix upright assert.

File: upright_asset/description/urdf/common/common.xacro (robot description, xacro)
@@ -2,5 +2,6 @@
 <robot xmlns:xacro="http://ros.org/wiki/xacro">
     <!-- Macro for creating links -->
-    <xacro:macro name="create_link" params="name mass ixx ixy ixz iyy iyz izz mesh_file material_name">
+    <xacro:macro name="create_link"
+                 params="name mass ixx ixy ixz iyy iyz izz mesh_file material_name scale='1 1 1' origin_xyz='0 0 0' origin_rpy='0 0 0' ">
         <link name="${name}">
             <inertial>
@@ -10,14 +11,14 @@
             </inertial>
             <visual>
-                <origin xyz="0 0 0" rpy="0 0 0"/>
+                <origin xyz="${origin_xyz}" rpy="${origin_rpy}"/>
                 <geometry>
-                    <mesh filename="${mesh_file}"/>
+                    <mesh filename="${mesh_file}" scale="${scale}"/>
                 </geometry>
                 <material name="${material_name}"/>
             </visual>
             <collision>
-                <origin xyz="0 0 0" rpy="0 0 0"/>
+                <origin xyz="${origin_xyz}" rpy="${origin_rpy}"/>
                 <geometry>
-                    <mesh filename="${mesh_file}"/>
+                    <mesh filename="${mesh_file}" scale="${scale}"/>
                 </geometry>
             </collision>
@@ -25,12 +26,13 @@
     </xacro:macro>
     <!-- Macro for creating joints with optional limits -->
-    <xacro:macro name="create_joint" params="name type parent child origin_xyz origin_rpy axis_xyz lower='0' upper='0' effort='0' velocity='0'">
+    <xacro:macro name="create_joint"
+                 params="name type parent child origin_xyz origin_rpy axis_xyz='0 0 1' lower='0' upper='0' effort='0' velocity='0'">
         <joint name="${name}" type="${type}">
             <origin xyz="${origin_xyz}" rpy="${origin_rpy}"/>
             <parent link="${parent}"/>
             <child link="${child}"/>
-            <axis xyz="${axis_xyz}"/>
             <!-- Conditionally add limits for revolute joints -->
             <xacro:if value="${type == 'revolute'}">
+                <axis xyz="${axis_xyz}"/>
                 <limit lower="${lower}" upper="${upper}" effort="${effort}" velocity="${velocity}"/>
             </xacro:if>

File: upright_asset/description/urdf/manipulator/qz_arm.xacro (robot description, xacro)
@@ -2,34 +2,38 @@
 <robot xmlns:xacro="http://ros.org/wiki/xacro" name="qz_arm">
     <!-- Include predefined materials -->
-    <!--    <xacro:include filename="$(find mm_assets)/description/urdf/common/materials.xacro"/>-->
-    <xacro:include filename="$(find mm_assets)/description/ddt_mm/urdf/common/common.xacro"/>
+    <!--    <xacro:include filename="$(find upright_asset)/description/urdf/common/materials.xacro"/>-->
+    <xacro:include filename="$(find upright_asset)/description/urdf/common/common.xacro"/>
     <!-- Link Definitions -->
     <xacro:create_link name="arm_base_link" mass="0.775915" ixx="0.000699851" ixy="5.34515E-06" ixz="1.76381E-06"
                        iyy="0.000855522" iyz="3.90737E-06" izz="0.00105822"
-                       mesh_file="package://mm_assets/description/ddt_mm/meshes/manipulator/base_link.STL"
+                       mesh_file="package://upright_asset/description/meshes/manipulator/base_link.STL"
                        material_name="grey"/>
     <xacro:create_link name="link1" mass="0.557107" ixx="0.000301325" ixy="-2.99504E-07" ixz="4.81746E-07"
                        iyy="0.000250218" iyz="1.49548E-05" izz="0.000325679"
-                       mesh_file="package://mm_assets/description/ddt_mm/meshes/manipulator/link1.STL"
+                       mesh_file="package://upright_asset/description/meshes/manipulator/link1.STL"
                        material_name="grey"/>
     <xacro:create_link name="link2" mass="0.646249" ixx="0.000351883" ixy="-7.83179E-05" ixz="8.22451E-05"
                        iyy="0.0019526" iyz="1.74745E-05" izz="0.00195686"
-                       mesh_file="package://mm_assets/description/ddt_mm/meshes/manipulator/link2.STL"
+                       mesh_file="package://upright_asset/description/meshes/manipulator/link2.STL"
                        material_name="grey"/>
     <xacro:create_link name="link3" mass="0.445563" ixx="0.00016737" ixy="-4.81066E-07" ixz="1.7795E-06"
                        iyy="0.000672323" iyz="-9.83781E-08" izz="0.000686599"
-                       mesh_file="package://mm_assets/description/ddt_mm/meshes/manipulator/link3.STL"
+                       mesh_file="package://upright_asset/description/meshes/manipulator/link3.STL"
                        material_name="grey"/>
     <xacro:create_link name="link4" mass="0.345885" ixx="0.000133803" ixy="-7.29532E-09" ixz="-2.46488E-07"
                        iyy="0.000121205" iyz="9.89248E-10" izz="0.00012501"
-                       mesh_file="package://mm_assets/description/ddt_mm/meshes/manipulator/link4.STL"
+                       mesh_file="package://upright_asset/description/meshes/manipulator/link4.STL"
                        material_name="grey"/>
     <xacro:create_link name="link5" mass="0.186636" ixx="0.000101781" ixy="-1.53593E-08" ixz="5.24141E-08"
                        iyy="8.27871E-05" iyz="-1.71996E-08" izz="8.59348E-05"
-                       mesh_file="package://mm_assets/description/ddt_mm/meshes/manipulator/link5.STL"
+                       mesh_file="package://upright_asset/description/meshes/manipulator/link5.STL"
                        material_name="grey"/>
     <xacro:create_link name="link6" mass="0.174621" ixx="5.00435E-05" ixy="0" ixz="0" iyy="5.00435E-05" iyz="0"
-                       izz="3.8504E-05" mesh_file="package://mm_assets/description/ddt_mm/meshes/manipulator/link6.STL"
+                       izz="3.8504E-05" mesh_file="package://upright_asset/description/meshes/manipulator/link6.STL"
                        material_name="grey"/>
+    <!--    <xacro:create_link name="Ee" mass="0.174621" ixx="5.00435E-05" ixy="0" ixz="0" iyy="5.00435E-05" iyz="0"-->
+    <!--                       izz="3.8504E-05" mesh_file="package://upright_asset/description/meshes/manipulator/Ee.stl"-->
+    <!--                       material_name="grey" origin_xyz="-0.04 0 0.04" origin_rpy="3.14 0 -1.57"-->
+    <!--                       scale="0.001 0.001 0.001"/>-->
     <!-- Joint Definitions -->
     <xacro:create_joint name="joint1" type="revolute" parent="arm_base_link" child="link1" origin_xyz="0 0 0.1127"
@@ -50,3 +54,5 @@
                         origin_rpy="0 1.5708 0" axis_xyz="0 0 1" lower="-3.14" upper="3.14" effort="110"
                         velocity="110"/>
+    <!--    <xacro:create_joint name="Ee_fixed" type="fixed" parent="link6" child="Ee" origin_xyz="0.0 0 0.0"-->
+    <!--                        origin_rpy="0 0 0"/>-->
 </robot>

File: upright_asset/description/urdf/manipulator/robot.xacro (robot description, xacro)
@@ -2,5 +2,5 @@
 <robot xmlns:xacro="http://www.ros.org/wiki/xacro" name="robot">
     <xacro:arg name="robot_type" default="qz_arm"/>
-    <xacro:include filename="$(find mm_assets)/description/ddt_mm/urdf/manipulator/qz_arm.xacro"/>
-    <xacro:include filename="$(find mm_assets)/description/ddt_mm/urdf/manipulator/gazebo.xacro"/>
+    <xacro:include filename="$(find upright_asset)/description/urdf/manipulator/qz_arm.xacro"/>
+    <xacro:include filename="$(find upright_asset)/description/urdf/manipulator/gazebo.xacro"/>
 </robot>
