Commit message: Could work in rviz.

File: upright_asset/description/urdf/diablo_manipulator/robot.urdf (robot description, URDF)
Before this commit: robot diablo_manipulator, 18 links, 17 joints
Links:
- removed link link1
- removed link link2
- removed link link3
- removed link link4
- removed link link5
- removed link link6
- added link Link1, mass 0.593563443690403; collision mesh filename=package://upright_asset/description/meshes/RM65/link1.STL; visual mesh filename=package://upright_asset/description/meshes/RM65/link1.STL
- added link Link2, mass 0.864175046869043; collision mesh filename=package://upright_asset/description/meshes/RM65/link2.STL; visual mesh filename=package://upright_asset/description/meshes/RM65/link2.STL
- added link Link3, mass 0.289633681624654; collision mesh filename=package://upright_asset/description/meshes/RM65/link3.STL; visual mesh filename=package://upright_asset/description/meshes/RM65/link3.STL
- added link Link4, mass 0.239419768320061; collision mesh filename=package://upright_asset/description/meshes/RM65/link4.STL; visual mesh filename=package://upright_asset/description/meshes/RM65/link4.STL
- added link Link5, mass 0.218799761431678; collision mesh filename=package://upright_asset/description/meshes/RM65/link5.STL; visual mesh filename=package://upright_asset/description/meshes/RM65/link5.STL
- added link Link6, mass 0.0649018034311231; collision mesh filename=package://upright_asset/description/meshes/RM65/link6.STL; visual mesh filename=package://upright_asset/description/meshes/RM65/link6.STL
- link arm_base_link: mass 0.775915 -> 0.841070778135659; geometry collision mesh filename=package://upright_asset/description/meshes/RM65/base_link.S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; visual mesh filename=package://upright_asset/description/meshes/RM65/base_link.S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
- link diablo_base_link: geometry collision mesh filename=package://upright_asset/description/meshes/diablo/base_link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 scale=1 1 1; visual mesh filename=package://upright_asset/description/meshes/diablo/base_link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 scale=1 1 1
- link left_leg1: geometry collision mesh filename=package://upright_asset/description/meshes/diablo/left_leg1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 scale=1 1 1; visual mesh filename=package://upright_asset/description/meshes/diablo/left_leg1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 scale=1 1 1
- link left_leg2: geometry collision mesh filename=package://upright_asset/description/meshes/diablo/left_leg2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 scale=1 1 1; visual mesh filename=package://upright_asset/description/meshes/diablo/left_leg2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 scale=1 1 1
- link left_leg3: geometry collision mesh filename=package://upright_asset/description/meshes/diablo/left_leg3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 scale=1 1 1; visual mesh filename=package://upright_asset/description/meshes/diablo/left_leg3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 scale=1 1 1
- link left_motor: geometry collision mesh filename=package://upright_asset/description/meshes/diablo/left_moto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 scale=1 1 1; visual mesh filename=package://upright_asset/description/meshes/diablo/left_moto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 scale=1 1 1
- link left_wheel: geometry collision mesh filename=package://upright_asset/description/meshes/diablo/left_whee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 scale=1 1 1; visual mesh filename=package://upright_asset/description/meshes/diablo/left_whee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 scale=1 1 1
- link right_leg1: geometry collision mesh filename=package://upright_asset/description/meshes/diablo/right_leg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 scale=1 1 1; visual mesh filename=package://upright_asset/description/meshes/diablo/right_leg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 scale=1 1 1
- link right_leg2: geometry collision mesh filename=package://upright_asset/description/meshes/diablo/right_leg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 scale=1 1 1; visual mesh filename=package://upright_asset/description/meshes/diablo/right_leg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 scale=1 1 1
- link right_leg3: geometry collision mesh filename=package://upright_asset/description/meshes/diablo/right_leg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 scale=1 1 1; visual mesh filename=package://upright_asset/description/meshes/diablo/right_leg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 scale=1 1 1
- link right_motor: geometry collision mesh filename=package://upright_asset/description/meshes/diablo/right_mot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 scale=1 1 1; visual mesh filename=package://upright_asset/description/meshes/diablo/right_mot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 scale=1 1 1
- link right_wheel: geometry collision mesh filename=package://upright_asset/description/meshes/diablo/right_whe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 scale=1 1 1; visual mesh filename=package://upright_asset/description/meshes/diablo/right_whe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 scale=1 1 1
Joints:
- joint joint1: child link1 -> Link1; limit lower=-3.14 upper=3.14 effort=110 velocity=110 -> lower=-3.1 upper=3.1 effort=60 velocity=3.14; origin xyz=0 0 0.1127 rpy=0 0 0 -> xyz=0 0 0.2405 rpy=0 0 0
- joint joint2: child link2 -> Link2; limit lower=-2.96 upper=0.17 effort=110 velocity=110 -> lower=-2.268 upper=2.268 effort=60 velocity=3.14; origin xyz=0 0 0 rpy=-1.5708 -0.38678 3.1416 -> xyz=0 0 0 rpy=1.5708 -1.5708 0; parent link1 -> Link1
- joint joint3: child link3 -> Link3; limit lower=-0.087 upper=3.14 effort=110 velocity=110 -> lower=-2.355 upper=2.355 effort=30 velocity=3.92; origin xyz=0.27009 1.3718E-05 0 rpy=0 0 -2.7548 -> xyz=0.256 0 0 rpy=0 0 1.5708; parent link2 -> Link2
- joint joint4: child link4 -> Link4; limit lower=-2.96 upper=2.96 effort=110 velocity=110 -> lower=-3.1 upper=3.1 effort=10 velocity=3.92; origin xyz=0.30854 0.0027492 0.00019049 rpy=-1.5708 0 -1.5708 -> xyz=0 -0.21 0 rpy=1.5708 0 0; parent link3 -> Link3
- joint joint5: child link5 -> Link5; limit lower=-1.74 upper=1.74 effort=110 velocity=110 -> lower=-2.233 upper=2.233 effort=10 velocity=3.92; origin xyz=0 0 0 rpy=0 -1.5708 0 -> xyz=0 0 0 rpy=-1.5708 0 0; parent link4 -> Link4
- joint joint6: child link6 -> Link6; limit lower=-3.14 upper=3.14 effort=110 velocity=110 -> lower=-6.28 upper=6.28 effort=10 velocity=3.92; origin xyz=0.0865 0 -0.0027486 rpy=0 1.5708 0 -> xyz=0 -0.144 0 rpy=1.5708 0 0; parent link5 -> Link5
- joint left_j1: axis 0 0 -1 -> (none)
- joint left_j2: axis 0 0 1 -> (none)
- joint left_j3: axis 0 0 -1 -> (none)
- joint left_j4: axis 0 0 -1 -> (none)
- joint left_j5: axis 0 0 1 -> (none)
- joint manipulator_joint: origin xyz=0.0 0.0 0.1 rpy=0.0 0.0 0.0 -> xyz=0.0 0.0 0.1 rpy=0.0 0.0 3.14
- joint right_j1: axis 0 0 -1 -> (none)
- joint right_j2: axis 0 0 1 -> (none)
- joint right_j3: axis 0 0 -1 -> (none)
- joint right_j4: axis 0 0 -1 -> (none)
- joint right_j5: axis 0 0 1 -> (none)

File: upright_asset/description/urdf/diablo_manipulator/robot.xacro (robot description, xacro)
@@ -8,5 +8,5 @@
         <parent link="diablo_base_link"/>
         <child link="arm_base_link"/>
-        <origin xyz="0.0 0.0 0.1" rpy="0.0 0.0 0.0"/>
+        <origin xyz="0.0 0.0 0.1" rpy="0.0 0.0 3.14"/>
     </joint>
     <gazebo>

File: upright_asset/description/urdf/diablo_manipulator/robot_pinocchio.urdf (robot description, URDF)
Before this commit: robot qm, 19 links, 18 joints
Links:
- removed link Ee_tray
- removed link link1
- removed link link2
- removed link link3
- removed link link4
- removed link link5
- removed link link6
- added link Link1, mass 0.593563443690403; collision mesh filename=package://upright_asset/description/meshes/RM65/link1.STL; visual mesh filename=package://upright_asset/description/meshes/RM65/link1.STL
- added link Link2, mass 0.864175046869043; collision mesh filename=package://upright_asset/description/meshes/RM65/link2.STL; visual mesh filename=package://upright_asset/description/meshes/RM65/link2.STL
- added link Link3, mass 0.289633681624654; collision mesh filename=package://upright_asset/description/meshes/RM65/link3.STL; visual mesh filename=package://upright_asset/description/meshes/RM65/link3.STL
- added link Link4, mass 0.239419768320061; collision mesh filename=package://upright_asset/description/meshes/RM65/link4.STL; visual mesh filename=package://upright_asset/description/meshes/RM65/link4.STL
- added link Link5, mass 0.218799761431678; collision mesh filename=package://upright_asset/description/meshes/RM65/link5.STL; visual mesh filename=package://upright_asset/description/meshes/RM65/link5.STL
- added link Link6, mass 0.0649018034311231; collision mesh filename=package://upright_asset/description/meshes/RM65/link6.STL; visual mesh filename=package://upright_asset/description/meshes/RM65/link6.STL
- link arm_base_link: mass 0.775915 -> 0.841070778135659; geometry collision mesh filename=package://upright_asset/description/meshes/RM65/base_link.S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; visual mesh filename=package://upright_asset/description/meshes/RM65/base_link.S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
- link diablo_base_link: geometry collision mesh filename=package://upright_asset/description/meshes/diablo/base_link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 scale=1 1 1; visual mesh filename=package://upright_asset/description/meshes/diablo/base_link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 scale=1 1 1
- link left_leg1: geometry collision mesh filename=package://upright_asset/description/meshes/diablo/left_leg1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 scale=1 1 1; visual mesh filename=package://upright_asset/description/meshes/diablo/left_leg1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 scale=1 1 1
- link left_leg2: geometry collision mesh filename=package://upright_asset/description/meshes/diablo/left_leg2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 scale=1 1 1; visual mesh filename=package://upright_asset/description/meshes/diablo/left_leg2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 scale=1 1 1
- link left_leg3: geometry collision mesh filename=package://upright_asset/description/meshes/diablo/left_leg3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 scale=1 1 1; visual mesh filename=package://upright_asset/description/meshes/diablo/left_leg3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 scale=1 1 1
- link left_motor: geometry collision mesh filename=package://upright_asset/description/meshes/diablo/left_moto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 scale=1 1 1; visual mesh filename=package://upright_asset/description/meshes/diablo/left_moto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 scale=1 1 1
- link left_wheel: geometry collision mesh filename=package://upright_asset/description/meshes/diablo/left_whee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 scale=1 1 1; visual mesh filename=package://upright_asset/description/meshes/diablo/left_whee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 scale=1 1 1
- link right_leg1: geometry collision mesh filename=package://upright_asset/description/meshes/diablo/right_leg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 scale=1 1 1; visual mesh filename=package://upright_asset/description/meshes/diablo/right_leg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 scale=1 1 1
- link right_leg2: geometry collision mesh filename=package://upright_asset/description/meshes/diablo/right_leg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 scale=1 1 1; visual mesh filename=package://upright_asset/description/meshes/diablo/right_leg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 scale=1 1 1
- link right_leg3: geometry collision mesh filename=package://upright_asset/description/meshes/diablo/right_leg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 scale=1 1 1; visual mesh filename=package://upright_asset/description/meshes/diablo/right_leg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 scale=1 1 1
- link right_motor: geometry collision mesh filename=package://upright_asset/description/meshes/diablo/right_mot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 scale=1 1 1; visual mesh filename=package://upright_asset/description/meshes/diablo/right_mot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 scale=1 1 1
- link right_wheel: geometry collision mesh filename=package://upright_asset/description/meshes/diablo/right_whe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 scale=1 1 1; visual mesh filename=package://upright_asset/description/meshes/diablo/right_whe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 scale=1 1 1
Joints:
- removed joint fix_Ee
- joint joint1: child link1 -> Link1; limit lower=-3.14 upper=3.14 effort=110 velocity=110 -> lower=-3.1 upper=3.1 effort=60 velocity=3.14; origin xyz=0 0 0.1127 rpy=0 0 0 -> xyz=0 0 0.2405 rpy=0 0 0
- joint joint2: child link2 -> Link2; limit lower=-2.96 upper=0.17 effort=110 velocity=110 -> lower=-2.268 upper=2.268 effort=60 velocity=3.14; origin xyz=0 0 0 rpy=-1.5708 -0.38678 3.1416 -> xyz=0 0 0 rpy=1.5708 -1.5708 0; parent link1 -> Link1
- joint joint3: child link3 -> Link3; limit lower=-0.087 upper=3.14 effort=110 velocity=110 -> lower=-2.355 upper=2.355 effort=30 velocity=3.92; origin xyz=0.27009 1.3718E-05 0 rpy=0 0 -2.7548 -> xyz=0.256 0 0 rpy=0 0 1.5708; parent link2 -> Link2
- joint joint4: child link4 -> Link4; limit lower=-2.96 upper=2.96 effort=110 velocity=110 -> lower=-3.1 upper=3.1 effort=10 velocity=3.92; origin xyz=0.30854 0.0027492 0.00019049 rpy=-1.5708 0 -1.5708 -> xyz=0 -0.21 0 rpy=1.5708 0 0; parent link3 -> Link3
- joint joint5: child link5 -> Link5; limit lower=-1.74 upper=1.74 effort=110 velocity=110 -> lower=-2.233 upper=2.233 effort=10 velocity=3.92; origin xyz=0 0 0 rpy=0 -1.5708 0 -> xyz=0 0 0 rpy=-1.5708 0 0; parent link4 -> Link4
- joint joint6: child link6 -> Link6; limit lower=-3.14 upper=3.14 effort=110 velocity=110 -> lower=-6.28 upper=6.28 effort=10 velocity=3.92; origin xyz=0.0865 0 -0.0027486 rpy=0 1.5708 0 -> xyz=0 -0.144 0 rpy=1.5708 0 0; parent link5 -> Link5
- joint manipulator_joint: origin xyz=0.0 0.0 0.1 rpy=0.0 0.0 0.0 -> xyz=0.0 0.0 0.1 rpy=0.0 0.0 3.14

File: upright_asset/description/urdf/manipulator/rm_65.urdf.xacro (robot description, xacro)
@@ -1,6 +1,6 @@
 <?xml version="1.0" encoding="utf-8"?>
 <robot name="rm_65" xmlns:xacro="http://www.ros.org/wiki/xacro">
-    <xacro:include filename="$(find upright_asset/description)/urdf/RM65/rm_65.transmission.xacro"/>
-    <xacro:include filename="$(find upright_asset/description)/urdf/RM65/rm_65.gazebo.xacro"/>
+    <xacro:include filename="$(find upright_asset)/description/urdf/manipulator/rm_65.transmission.xacro"/>
+    <xacro:include filename="$(find upright_asset)/description/urdf/manipulator/rm_65.gazebo.xacro"/>
     <!-- Inertial matrix -->
     <xacro:macro name="inertial_matrix" params="mass">
@@ -18,30 +18,6 @@
         </inertial>
     </xacro:macro>
-    <link name="dummy">
-    </link>
     <!-- ///////////////////////////////////////   bottom_joint   ////////////////////////////////////////// -->
-    <joint name="bottom_joint" type="fixed">
-        <origin xyz="0 0 0" rpy="0 0 0"/>
-        <parent link="base_link"/>
-        <child link="bottom_link"/>
-    </joint>
-    <link name="bottom_link">
-        <visual>
-            <origin xyz=" 0 0 -0.02" rpy="0 0 0"/>
-            <geometry>
-                <box size="0.06 0.06 0.02"/>
-            </geometry>
-            <material name="Brown"/>
-        </visual>
-        <collision>
-            <origin xyz=" 0 0 0" rpy="0 0 0"/>
-            <geometry>
-                <box size="0.06 0.06 0.02"/>
-            </geometry>
-        </collision>
-        <xacro:Box_inertial_matrix m="500" l="1" w="1" h="0.02"/>
-    </link>
-    <link
-            name="base_link">
+    <link name="arm_base_link">
         <inertial>
             <origin
@@ -82,16 +58,5 @@
         </collision>
     </link>
-    <gazebo reference="base_link">
-        <mu1 value="200000.0"/>
-        <mu2 value="200000.0"/>
-        <kp value="100000000.0"/>
-        <kd value="1.0"/>
-    </gazebo>
-    <joint name="dummy_joint" type="fixed">
-        <parent link="dummy"/>
-        <child link="base_link"/>
-    </joint>
-    <link
-            name="Link1">
+    <link name="Link1">
         <inertial>
             <origin
@@ -132,12 +97,11 @@
         </collision>
     </link>
-    <joint
-            name="joint1"
-            type="revolute">
+    <joint name="joint1"
+           type="revolute">
         <origin
                 xyz="0 0 0.2405"
                 rpy="0 0 0"/>
         <parent
-                link="base_link"/>
+                link="arm_base_link"/>
         <child
                 link="Link1"/>

File: upright_asset/description/urdf/manipulator/robot.xacro (robot description, xacro)
@@ -1,5 +1,5 @@
 <?xml version="1.0"?>
 <robot xmlns:xacro="http://www.ros.org/wiki/xacro" name="robot">
-    <xacro:arg name="robot_type" default="rm_a65"/>
+    <xacro:arg name="robot_type" default="rm_65"/>
     <xacro:include filename="$(find upright_asset)/description/urdf/manipulator/rm_65.urdf.xacro"/>
 </robot>
