Commit message: Change manipulator urdf and meshes.

File: upright_asset/description/urdf/diablo_manipulator/robot.xacro (robot description, xacro)
@@ -1,4 +1,4 @@
 <?xml version="1.0"?>
-<robot xmlns:xacro="http://www.ros.org/wiki/xacro" name="qm">
+<robot xmlns:xacro="http://www.ros.org/wiki/xacro" name="wlm">
     <xacro:arg name="robot_type" default="ddt"/>
     <xacro:include filename="$(find upright_asset)/description/urdf/diablo/robot.xacro"/>
@@ -8,5 +8,5 @@
         <parent link="diablo_base_link"/>
         <child link="arm_base_link"/>
-        <origin xyz="0.0 0.0 0.1" rpy="0.0 0.0 3.14"/>
+        <origin xyz="0.0 0.0 0.1" rpy="0.0 0.0 0.0"/>
     </joint>
     <gazebo>

File: upright_asset/description/urdf/manipulator/robot.xacro (robot description, xacro)
@@ -1,5 +1,5 @@
 <?xml version="1.0"?>
-<robot xmlns:xacro="http://www.ros.org/wiki/xacro" name="robot">
-    <xacro:arg name="robot_type" default="rm_65"/>
-    <xacro:include filename="$(find upright_asset)/description/urdf/manipulator/rm_65.urdf.xacro"/>
+<robot xmlns:xacro="http://ros.org/wiki/xacro" name="swingboy_v1">
+    <xacro:include filename="$(find upright_asset)/description/urdf/manipulator/arm.urdf.xacro"/>
+    <xacro:include filename="$(find upright_asset)/description/urdf/manipulator/gazebo.xacro"/>
 </robot>

Commit message: Could use fake.

File: upright_asset/description/urdf/diablo_manipulator/robot.xacro (robot description, xacro)
@@ -22,11 +22,3 @@
         </plugin>
     </gazebo>
-    <!-- ros_control plugin -->
-    <!--    <gazebo>-->
-    <!--        <plugin name="gazebo_ros_control" filename="libqm_hw_sim.so">-->
-    <!--            <robotNamespace>/</robotNamespace>-->
-    <!--            <robotParam>upright_asset</robotParam>-->
-    <!--            <robotSimType>qm_gazebo/QMHWSim</robotSimType>-->
-    <!--        </plugin>-->
-    <!--    </gazebo>-->
 </robot>

File: upright_asset/description/urdf/diablo_manipulator/robot_pinocchio.urdf (robot description, URDF)
Before this commit: robot diablo_rm, 18 links, 17 joints
Links:
- removed link Link1
- removed link Link2
- removed link Link3
- removed link Link4
- removed link Link5
- removed link Link6
- added link link1, mass 1.103721; collision mesh filename=package://upright_asset/description/meshes/manipulator/link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; visual mesh filename=package://upright_asset/description/meshes/manipulator/link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
- added link link2, mass 0.534276; collision mesh filename=package://upright_asset/description/meshes/manipulator/link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; visual mesh filename=package://upright_asset/description/meshes/manipulator/link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
- added link link3, mass 0.474451; collision mesh filename=package://upright_asset/description/meshes/manipulator/link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; visual mesh filename=package://upright_asset/description/meshes/manipulator/link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
- added link link4, mass 0.056678; collision mesh filename=package://upright_asset/description/meshes/manipulator/link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; visual mesh filename=package://upright_asset/description/meshes/manipulator/link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
- added link link5, mass 0.598593; collision mesh filename=package://upright_asset/description/meshes/manipulator/link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; visual mesh filename=package://upright_asset/description/meshes/manipulator/link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
- added link link6, mass 0.001; collision mesh filename=package://upright_asset/description/meshes/manipulator/link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; visual mesh filename=package://upright_asset/description/meshes/manipulator/link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
- link arm_base_link: mass 0.841070778135659 -> 6.722526; geometry collision mesh filename=package://upright_asset/description/meshes/manipulator/base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; visual mesh filename=package://upright_asset/description/meshes/manipulator/base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
Joints:
- joint joint1: child Link1 -> link1; limit lower=-3.1 upper=3.1 effort=60 velocity=3.14 -> lower=-1.57 upper=1.57 effort=150 velocity=1.5; origin xyz=0 0 0.2405 rpy=0 0 0 -> xyz=0 0 0.07925 rpy=0 0 0
- joint joint2: axis 0 0 1 -> 0 1 0; child Link2 -> link2; limit lower=-2.268 upper=2.268 effort=60 velocity=3.14 -> lower=0 upper=1.57 effort=150 velocity=1.5; origin xyz=0 0 0 rpy=1.5708 -1.5708 0 -> xyz=0 0 0.0365 rpy=0 0 0; parent Link1 -> link1
- joint joint3: axis 0 0 1 -> 0 1 0; child Link3 -> link3; limit lower=-2.355 upper=2.355 effort=30 velocity=3.92 -> lower=-1.57 upper=0 effort=150 velocity=1.5; origin xyz=0.256 0 0 rpy=0 0 1.5708 -> xyz=-0.220 0 0 rpy=0 0 0; parent Link2 -> link2
- joint joint4: axis 0 0 1 -> 0 1 0; child Link4 -> link4; limit lower=-3.1 upper=3.1 effort=10 velocity=3.92 -> lower=-1.5 upper=0.5 effort=150 velocity=1.5; origin xyz=0 -0.21 0 rpy=1.5708 0 0 -> xyz=0.220 0 0.057 rpy=0 0 0; parent Link3 -> link3
- joint joint5: child Link5 -> link5; limit lower=-2.233 upper=2.233 effort=10 velocity=3.92 -> lower=-0.785 upper=0.785 effort=150 velocity=1.5; origin xyz=0 0 0 rpy=-1.5708 0 0 -> xyz=0.0615 0 0.0825 rpy=0 0 0; parent Link4 -> link4
- joint joint6: axis 0 0 1 -> 1 0 0; child Link6 -> link6; limit lower=-6.28 upper=6.28 effort=10 velocity=3.92 -> lower=-1.57 upper=1.57 effort=150 velocity=1.5; origin xyz=0 -0.144 0 rpy=1.5708 0 0 -> xyz=0.0285 0 -0.0825 rpy=0 0 0; parent Link5 -> link5
- joint manipulator_joint: origin xyz=0.0 0.0 0.1 rpy=0.0 0.0 3.14 -> xyz=0.0 0.0 0.1 rpy=0.0 0.0 0.0
